Commit message: Properly add gazebo plugins to URDF.

File: models/sjtu_drone/sjtu_drone.urdf (robot description, URDF)
Before this commit: robot sjtu_drone, 1 links, 0 joints
Links:
- removed link sjtu_drone__base_link
- added link base_link, mass 1.477; collision mesh filename=package://sjtu_drone/models/sjtu_drone/quadrotor_4.dae scale=1.0 1.0 1.0; visual mesh filename=package://sjtu_drone/models/sjtu_drone/quadrotor_4.dae scale=1.0 1.0 1.0
